Commit message: fixes

File: Robots/h1_with_hand.urdf (robot description, URDF)
Before this commit: robot h1, 52 links, 51 joints
Joints:
- removed joint left_hand_joint
- removed joint right_hand_joint
- added joint left_wrist: type revolute, parent left_elbow_link, child left_hand_link, origin xyz=0.2605 0 -0.0185 rpy=0 0 0, axis 1 0 0, limit lower=-3.0543261909900767596164588448551 upper=3.0543261909900767596164588448551 effort=6 velocity=12
- added joint right_wrist: type revolute, parent right_elbow_link, child right_hand_link, origin xyz=0.2605 0 -0.0185 rpy=0 0 0, axis 1 0 0, limit lower=-3.0543261909900767596164588448551 upper=3.0543261909900767596164588448551 effort=6 velocity=12
